Commit message: updated cube sizes added put-in-green-cup task corrected missing preprocess in attention and transport

File: cliport/environments/assets/stacking/coffee_cube.urdf (robot description, URDF)
Before this commit: robot box.urdf, 1 links, 0 joints
Links:
- link baseLink: mass .1 -> .01; geometry collision box size=0.03 0.03 0.01; visual box size=0.03 0.03 0.01

File: cliport/environments/assets/stacking/sugar_cube.urdf (robot description, URDF)
Before this commit: robot box.urdf, 1 links, 0 joints
Links:
- link baseLink: mass .1 -> .01; geometry collision box size=0.04 0.04 0.01; visual box size=0.04 0.04 0.01
